Commit message: Prvy uspesny test hybania s ramenom cez moveit (v pritomnosti kolizneho objektu). Frekvencia 15Hz

File: scara_v2_with_gripper/urdf/scara_and_rt_urdf.xacro (robot description, xacro)
@@ -153,33 +153,33 @@
     </joint>
     <!--_______Colision object_______-->
-    <!--<link name="colisionBox">-->
-        <!--<inertial>-->
-            <!--<origin xyz="0 0 0" rpy="0 0 0" />-->
-            <!--<mass value="1" />-->
-            <!--<inertia ixx="1" ixy="0" ixz="0"-->
-                     <!--iyy="1" iyz="0"-->
-                     <!--izz="1" />-->
-        <!--</inertial>-->
-        <!--<visual>-->
-            <!--<origin xyz="0 0 0" rpy="0 0 0" />-->
-            <!--<geometry>-->
-                <!--<box size="0.05 0.05 0.2"/>-->
-            <!--</geometry>-->
-            <!--<material name="sensoSilver">-->
-            <!--</material>-->
-        <!--</visual>-->
-        <!--<collision>-->
-            <!--<origin xyz="0 0 0" rpy="0 0 0" />-->
-            <!--<geometry>-->
-                <!--<box size="0.1 0.1 0.2"/>-->
-            <!--</geometry>-->
-        <!--</collision>-->
-    <!--</link>-->
-    <!--<joint name="Joint_colisionBox" type="fixed">-->
-        <!--<parent link="BaseBox" />-->
-        <!--<child link="colisionBox" />-->
-        <!--<origin xyz="0.55 0.40 0.1" rpy="0 0 0" />-->
-        <!--<axis xyz="1 0 0" />-->
-    <!--</joint>-->
+    <link name="colisionBox">
+        <inertial>
+            <origin xyz="0 0 0" rpy="0 0 0" />
+            <mass value="1" />
+            <inertia ixx="1" ixy="0" ixz="0"
+                     iyy="1" iyz="0"
+                     izz="1" />
+        </inertial>
+        <visual>
+            <origin xyz="0 0 0" rpy="0 0 0" />
+            <geometry>
+                <box size="0.05 0.05 0.2"/>
+            </geometry>
+            <material name="red">
+            </material>
+        </visual>
+        <collision>
+            <origin xyz="0 0 0" rpy="0 0 0" />
+            <geometry>
+                <box size="0.1 0.1 0.2"/>
+            </geometry>
+        </collision>
+    </link>
+    <joint name="Joint_colisionBox" type="fixed">
+        <parent link="BaseBox" />
+        <child link="colisionBox" />
+        <origin xyz="0.55 0.40 0.1" rpy="0 0 0" />
+        <axis xyz="1 0 0" />
+    </joint>
     <!--**************************-->
     <link name="placeHole1">

Commit message: GUI - DEMO mode funguje aj ked pomaly..

File: scara_v2_with_gripper/urdf/scara_and_rt_urdf.xacro (robot description, xacro)
@@ -172,5 +172,5 @@
             <origin xyz="0 0 0" rpy="0 0 0" />
             <geometry>
-                <box size="0.1 0.1 0.2"/>
+                <box size="0.07 0.07 0.2"/>
             </geometry>
         </collision>
@@ -440,10 +440,10 @@
             <material name="sensoBlack" />
         </visual>
-        <collision>
-            <origin xyz="0 0 0" rpy="0 0 0" />
-            <geometry>
-                <box size="0.15 0.1 0.02"/>
-            </geometry>
-        </collision>
+        <!--<collision>-->
+            <!--<origin xyz="0 0 0" rpy="0 0 0" />-->
+            <!--<geometry>-->
+                <!--<box size="0.15 0.1 0.01"/>-->
+            <!--</geometry>-->
+        <!--</collision>-->
     </link>
     <joint name="world_to_base" type="fixed">
@@ -468,10 +468,10 @@
             <material name="sensoSilver" />
         </visual>
-        <collision>
-            <origin xyz="0 0 0" rpy="0 0 0" />
-            <geometry>
-                <cylinder length="0.01" radius="0.02"/>
-            </geometry>
-        </collision>
+        <!--<collision>-->
+            <!--<origin xyz="0 0 0" rpy="0 0 0" />-->
+            <!--<geometry>-->
+                <!--<cylinder length="0.01" radius="0.02"/>-->
+            <!--</geometry>-->
+        <!--</collision>-->
     </link>
     <joint name="base_to_base_link1" type="fixed">
@@ -496,10 +496,10 @@
             <material name="sensoSilver" />
         </visual>
-        <collision>
-            <origin xyz="0 0 0" rpy="0 0 0" />
-            <geometry>
-                <cylinder length="0.02" radius="0.06"/>
-            </geometry>
-        </collision>
+        <!--<collision>-->
+            <!--<origin xyz="0 0 0" rpy="0 0 0" />-->
+            <!--<geometry>-->
+                <!--<cylinder length="0.01" radius="0.06"/>-->
+            <!--</geometry>-->
+        <!--</collision>-->
     </link>
     <joint name="base_link1_to_link1" type="revolute"> <!-- rotary table joint-->
@@ -525,10 +525,10 @@
             <material name="blue" />
         </visual>
-        <collision>
-            <origin xyz="0 0 0" rpy="0 0 0" />
-            <geometry>
-                <cylinder length="0.005" radius="0.01"/>
-            </geometry>
-        </collision>
+        <!--<collision>-->
+            <!--<origin xyz="0 0 0" rpy="0 0 0" />-->
+            <!--<geometry>-->
+                <!--<cylinder length="0.005" radius="0.01"/>-->
+            <!--</geometry>-->
+        <!--</collision>-->
     </link>
     <joint name="link1_to_hole1" type="fixed">
@@ -552,10 +552,10 @@
             <material name="white" />
         </visual>
-        <collision>
-            <origin xyz="0 0 0" rpy="0 0 0" />
-            <geometry>
-                <cylinder length="0.005" radius="0.01"/>
-            </geometry>
-        </collision>
+        <!--<collision>-->
+            <!--<origin xyz="0 0 0" rpy="0 0 0" />-->
+            <!--<geometry>-->
+                <!--<cylinder length="0.005" radius="0.01"/>-->
+            <!--</geometry>-->
+        <!--</collision>-->
     </link>
     <joint name="link1_to_hole8" type="fixed">
@@ -579,10 +579,10 @@
             <material name="white" />
         </visual>
-        <collision>
-            <origin xyz="0 0 0" rpy="0 0 0" />
-            <geometry>
-                <cylinder length="0.005" radius="0.01"/>
-            </geometry>
-        </collision>
+        <!--<collision>-->
+            <!--<origin xyz="0 0 0" rpy="0 0 0" />-->
+            <!--<geometry>-->
+                <!--<cylinder length="0.005" radius="0.01"/>-->
+            <!--</geometry>-->
+        <!--</collision>-->
     </link>
     <joint name="link1_to_hole7" type="fixed">
@@ -606,10 +606,10 @@
             <material name="white" />
         </visual>
-        <collision>
-            <origin xyz="0 0 0" rpy="0 0 0" />
-            <geometry>
-                <cylinder length="0.005" radius="0.01"/>
-            </geometry>
-        </collision>
+        <!--<collision>-->
+            <!--<origin xyz="0 0 0" rpy="0 0 0" />-->
+            <!--<geometry>-->
+                <!--<cylinder length="0.005" radius="0.01"/>-->
+            <!--</geometry>-->
+        <!--</collision>-->
     </link>
     <joint name="link1_to_hole6" type="fixed">
@@ -633,10 +633,10 @@
             <material name="white" />
         </visual>
-        <collision>
-            <origin xyz="0 0 0" rpy="0 0 0" />
-            <geometry>
-                <cylinder length="0.005" radius="0.01"/>
-            </geometry>
-        </collision>
+        <!--<collision>-->
+            <!--<origin xyz="0 0 0" rpy="0 0 0" />-->
+            <!--<geometry>-->
+                <!--<cylinder length="0.005" radius="0.01"/>-->
+            <!--</geometry>-->
+        <!--</collision>-->
     </link>
     <joint name="link1_to_hole5" type="fixed">
@@ -660,10 +660,10 @@
             <material name="white" />
         </visual>
-        <collision>
-            <origin xyz="0 0 0" rpy="0 0 0" />
-            <geometry>
-                <cylinder length="0.005" radius="0.01"/>
-            </geometry>
-        </collision>
+        <!--<collision>-->
+            <!--<origin xyz="0 0 0" rpy="0 0 0" />-->
+            <!--<geometry>-->
+                <!--<cylinder length="0.005" radius="0.01"/>-->
+            <!--</geometry>-->
+        <!--</collision>-->
     </link>
     <joint name="link1_to_hole4" type="fixed">
@@ -687,10 +687,10 @@
             <material name="white" />
         </visual>
-        <collision>
-            <origin xyz="0 0 0" rpy="0 0 0" />
-            <geometry>
-                <cylinder length="0.005" radius="0.01"/>
-            </geometry>
-        </collision>
+        <!--<collision>-->
+            <!--<origin xyz="0 0 0" rpy="0 0 0" />-->
+            <!--<geometry>-->
+                <!--<cylinder length="0.005" radius="0.01"/>-->
+            <!--</geometry>-->
+        <!--</collision>-->
     </link>
     <joint name="link1_to_hole3" type="fixed">
@@ -714,10 +714,10 @@
             <material name="white" />
         </visual>
-        <collision>
-            <origin xyz="0 0 0" rpy="0 0 0" />
-            <geometry>
-                <cylinder length="0.005" radius="0.01"/>
-            </geometry>
-        </collision>
+        <!--<collision>-->
+            <!--<origin xyz="0 0 0" rpy="0 0 0" />-->
+            <!--<geometry>-->
+                <!--<cylinder length="0.005" radius="0.01"/>-->
+            <!--</geometry>-->
+        <!--</collision>-->
     </link>
     <joint name="link1_to_hole2" type="fixed">
