Commit message: SENSODRIVE 27.Apr.2018 - FINAL COMMIT!!!!!

File: gazebo_scara_and_rt/scara_v2_full_description/urdf/scara_and_rt_v3_urdf.xacro (robot description, xacro)
@@ -757,5 +757,5 @@
         <actuator name="motor1">
             <hardwareInterface>hardware_interface/EffortJointInterface</hardwareInterface>
-            <mechanicalReduction>1</mechanicalReduction>
+            <mechanicalReduction>101</mechanicalReduction>
         </actuator>
     </transmission>
@@ -767,5 +767,5 @@
         <actuator name="motor2">
             <hardwareInterface>hardware_interface/EffortJointInterface</hardwareInterface>
-            <mechanicalReduction>1</mechanicalReduction>
+            <mechanicalReduction>101</mechanicalReduction>
         </actuator>
     </transmission>

File: scara_v2_with_gripper/urdf/scara_and_rt_v3_urdf.xacro (robot description, xacro)
@@ -6,5 +6,5 @@
     <xacro:property name="M_PI" value="3.141592" />
     <xacro:property name="baseBox_offset_x" value="0.4" />
-    <xacro:property name="baseBox_offset_y" value="0.15" />
+    <xacro:property name="baseBox_offset_y" value="0.25" />
     <xacro:property name="base_size_x" value="0.125" />
     <xacro:property name="base_size_y" value="0.245" />
@@ -400,5 +400,5 @@
                 <box size="${base_size_x} ${base_size_y} ${base_size_z}"/>
             </geometry>
-            <material name="sensoGray" />
+            <material name="sensoSilver" />
         </visual>
         <collision>
@@ -681,10 +681,10 @@
         <limit effort="100.0" lower="-0.04" upper="0.05" velocity="1"/>
     </joint>
-    <!--<joint name="Base_to_tool0" type="fixed">-->
-    <!--<parent link="GripperBase" />-->
-    <!--<child link="tool0" />-->
-    <!--<origin xyz="0 0.0984 0" rpy="0 0 0 " />-->
-    <!--</joint>-->
-    <!--<link name="tool0"/>-->
+    <joint name="Base_to_tool0" type="fixed">
+    <parent link="GripperBase" />
+    <child link="tool0" />
+    <origin xyz="0 0.0984 0" rpy="0 0 0 " />
+    </joint>
+    <link name="tool0"/>
     <link name="GripperLeft">
         <inertial>
